File: Bruno Drink Machine/EAGLE files/LCD Board/LCD ctrl.sch (EAGLE design)
At the start: 32 parts, among them IC1 PIC24FJ256DA210-I/PT, IC2 IS62LV256AL, IC3 IS62LV256AL, IC4 BA3259H-HRP5, P1 CONN-40P-62684-401100ALF, P18 CONN-8P-PND, P2 USB-CON690-005-299-043

Commit message: made some of the changes; not all (will need to go through change list and confirm later)
Changed lines of the file:
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@@
 <?xml version="1.0" encoding="utf-8"?>
 <!DOCTYPE eagle SYSTEM "eagle.dtd">
-<eagle version="8.2.2">
+<eagle version="9.2.2">
 <drawing>
 <settings>
 <setting alwaysvectorfont="yes"/>
+<setting keepoldvectorfont="yes"/>
 <setting verticaltext="up"/>
 </settings>
@@
 <layer number="91" name="Nets" color="2" fill="1" visible="yes" active="yes"/>
 <layer number="92" name="Busses" color="1" fill="1" visible="yes" active="yes"/>
-<layer number="93" name="Pins" color="2" fill="1" visible="no" active="yes"/>
+<layer number="93" name="Pins" color="2" fill="1" visible="yes" active="yes"/>
 <layer number="94" name="Symbols" color="4" fill="1" visible="yes" active="yes"/>
 <layer number="95" name="Names" color="7" fill="1" visible="yes" active="yes"/>
-<layer number="96" name="Values" color="7" fill="1" visible="no" active="yes"/>
+<layer number="96" name="Values" color="7" fill="1" visible="yes" active="yes"/>
 <layer number="97" name="Info" color="7" fill="1" visible="yes" active="yes"/>
 <layer number="98" name="Guide" color="6" fill="1" visible="yes" active="yes"/>
@@
 <wire x1="22.86" y1="111.76" x2="20.32" y2="111.76" width="0.1524" layer="91"/>
 <wire x1="20.32" y1="111.76" x2="20.32" y2="73.66" width="0.1524" layer="91"/>
-</segment>
-<segment>
+<label x="5.08" y="109.22" size="1.778" layer="95"/>
+</segment>
+<segment>
