File: Bruno Drink Machine/EAGLE files/LCD Board/LCD ctrl.sch (EAGLE design)
At the start: 32 parts, among them IC1 PIC24FJ256DA210-I/PT, IC2 IS62LV256AL, IC3 IS62LV256AL, IC4 BA3259H-HRP5, P1 CONN-40P-62684-401100ALF, P18 CONN-8P-PND, P2 USB-CON690-005-299-043

Commit message: commit before merge
Parts:
- renumbered P18 to P3
Changed lines of the file:
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@@
 <layer number="94" name="Symbols" color="4" fill="1" visible="yes" active="yes"/>
 <layer number="95" name="Names" color="7" fill="1" visible="yes" active="yes"/>
-<layer number="96" name="Values" color="7" fill="1" visible="no" active="yes"/>
+<layer number="96" name="Values" color="7" fill="1" visible="yes" active="yes"/>
 <layer number="97" name="Info" color="7" fill="1" visible="yes" active="yes"/>
 <layer number="98" name="Guide" color="6" fill="1" visible="yes" active="yes"/>
@@
 <part name="IC1" library="Aaron SMT" deviceset="PIC24FJ256DA210" device="-I/PT"/>
 <part name="P1" library="Aaron SMT" deviceset="CONN-40P" device="-62684-401100ALF"/>
-<part name="P18" library="Aaron" deviceset="CONN-8P" device="-PND"/>
+<part name="P3" library="Aaron" deviceset="CONN-8P" device="-PND"/>
 <part name="U$26" library="Aaron" deviceset="GND" device=""/>
 <part name="U$1" library="Aaron" deviceset="GND" device=""/>
@@
 <attribute name="NAME" x="142.24" y="-30.48" size="1.778" layer="95"/>
 </instance>
-<instance part="P18" gate="P" x="147.32" y="66.04" smashed="yes" rot="MR0">
+<instance part="P3" gate="P" x="147.32" y="66.04" smashed="yes" rot="MR0">
 <attribute name="NAME" x="149.86" y="48.26" size="1.27" layer="95" rot="MR0"/>
 </instance>
@@
 <net name="GND" class="0">
 <segment>
-<pinref part="P18" gate="P" pin="3"/>
+<pinref part="P3" gate="P" pin="3"/>
 <pinref part="U$26" gate="GND" pin="GND"/>
 <wire x1="144.78" y1="63.5" x2="142.24" y2="63.5" width="0.1524" layer="91"/>
@@
 <net name="12V" class="0">
 <segment>
-<pinref part="P18" gate="P" pin="1"/>
+<pinref part="P3" gate="P" pin="1"/>
 <wire x1="144.78" y1="68.58" x2="142.24" y2="68.58" width="0.1524" layer="91"/>
 <wire x1="142.24" y1="68.58" x2="142.24" y2="73.66" width="0.1524" layer="91"/>
@@
 <net name="MOSI" class="0">
 <segment>
-<pinref part="P18" gate="P" pin="5"/>
+<pinref part="P3" gate="P" pin="5"/>
 <wire x1="144.78" y1="58.42" x2="137.16" y2="58.42" width="0.1524" layer="91"/>
 <label x="132.08" y="58.42" size="1.778" layer="95"/>
@@
 <net name="SCK" class="0">
 <segment>
-<pinref part="P18" gate="P" pin="7"/>
+<pinref part="P3" gate="P" pin="7"/>
 <wire x1="144.78" y1="53.34" x2="137.16" y2="53.34" width="0.1524" layer="91"/>
 <label x="132.08" y="53.34" size="1.778" layer="95"/>
@@
 <net name="!SS" class="0">
 <segment>
-<pinref part="P18" gate="P" pin="8"/>
+<pinref part="P3" gate="P" pin="8"/>
 <wire x1="144.78" y1="50.8" x2="137.16" y2="50.8" width="0.1524" layer="91"/>
 <label x="132.08" y="50.8" size="1.778" layer="95"/>
@@
 <net name="MISO" class="0">
 <segment>
-<pinref part="P18" gate="P" pin="6"/>
+<pinref part="P3" gate="P" pin="6"/>
 <wire x1="144.78" y1="55.88" x2="137.16" y2="55.88" width="0.1524" layer="91"/>
 <label x="132.08" y="55.88" size="1.778" layer="95"/>
@@
 <net name="+5V" class="1">
 <segment>
-<pinref part="P18" gate="P" pin="2"/>
+<pinref part="P3" gate="P" pin="2"/>
 <wire x1="144.78" y1="66.04" x2="134.62" y2="66.04" width="0.1524" layer="91"/>
 <wire x1="134.62" y1="66.04" x2="134.62" y2="73.66" width="0.1524" layer="91"/>
